File: Hardware/Eagle files/Smart ezNODE 503 M3.brd (EAGLE design)
At the start: 97.2 x 63.4 mm, 18 parts, among them K1 G6K-2F-Y, K2 G6K-2F-Y, Q1 MMBT5088, Q2 MMBT5088, X1 SSW-114-02-S-D-DH

Commit message: Add files via upload
Routing:
- net VCC33: track 61.1 -> 81.5 mm
- net N$1: track 16.6 -> 32.2 mm
- net N$2: track 16.7 -> 32.2 mm
- net EXT_OUT_1: track 67.6 -> 52.7 mm
- net N$16: track 45.6 -> 38.2 mm, vias 3 -> 1
- net N$4: track 22.0 -> 19.3 mm, vias 2 -> 1
- net N$12: track 24.4 -> 26.1 mm
- net N$19: track 25.3 -> 26.1 mm
- net N$3: track 11.2 -> 11.6 mm, vias 0 -> 1
