File: Hardware/Eagle files/Smart ezNODE 503 M3.sch (EAGLE design)
At the start: 18 parts, among them K1 G6K-2F-Y, K2 G6K-2F-Y, Q1 MMBT5088, Q2 MMBT5088, X1 SSW-114-02-S-D-DH

Commit message: Add files via upload
Connections:
- net VCC33: now also PWS1.+VOUT2/NC; no longer PWS1.+VOUT1
Changed lines of the file:
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@@
 <instances>
 <instance part="FRAME1" gate="G$1" x="0" y="0"/>
-<instance part="GND2" gate="1" x="213.36" y="213.36"/>
+<instance part="GND2" gate="1" x="223.52" y="213.36"/>
 <instance part="X1" gate="-1" x="181.61" y="69.85" smashed="yes" rot="MR0">
 <attribute name="VALUE" x="181.61" y="73.66" size="1.778" layer="96"/>
@@
 <instance part="X3" gate="-7" x="307.34" y="121.92"/>
 <instance part="X3" gate="-8" x="307.34" y="114.3"/>
-<instance part="PWS1" gate="G$1" x="193.04" y="218.44"/>
+<instance part="PWS1" gate="G$1" x="193.04" y="218.44" smashed="yes">
+<attribute name="NAME" x="182.88" y="227.33" size="1.778" layer="95"/>
+<attribute name="VALUE" x="182.88" y="207.01" size="1.778" layer="96"/>
+</instance>
 </instances>
 <busses>
@@
 <nets>
 <net name="VCC33" class="1">
-<segment>
-<wire x1="208.28" y1="220.98" x2="213.36" y2="220.98" width="0.1524" layer="91"/>
-<label x="215.9" y="220.98" size="1.27" layer="95"/>
-<pinref part="PWS1" gate="G$1" pin="+VOUT1"/>
-</segment>
 <segment>
 <pinref part="X1" gate="-2" pin="1"/>
@@
 <wire x1="283.21" y1="123.19" x2="283.21" y2="125.73" width="0.1524" layer="91"/>
 </segment>
+<segment>
+<wire x1="208.28" y1="215.9" x2="213.36" y2="215.9" width="0.1524" layer="91"/>
+<label x="215.9" y="215.9" size="1.27" layer="95"/>
+<pinref part="PWS1" gate="G$1" pin="+VOUT2/NC"/>
+</segment>
 </net>
 <net name="GND" class="1">
 <segment>
-<wire x1="208.28" y1="218.44" x2="213.36" y2="218.44" width="0.1524" layer="91"/>
-<wire x1="213.36" y1="218.44" x2="213.36" y2="215.9" width="0.1524" layer="91"/>
+<wire x1="208.28" y1="218.44" x2="223.52" y2="218.44" width="0.1524" layer="91"/>
+<wire x1="223.52" y1="218.44" x2="223.52" y2="215.9" width="0.1524" layer="91"/>
 <pinref part="GND2" gate="1" pin="GND"/>
 <pinref part="PWS1" gate="G$1" pin="COM"/>
@@
 </segment>
 </net>
-<net name="N$1" class="2">
+<net name="N$1" class="0">
 <segment>
 <pinref part="X2" gate="-1" pin="SK"/>
@@
 </segment>
 </net>
-<net name="N$2" class="2">
+<net name="N$2" class="0">
 <segment>
 <pinref part="X2" gate="-2" pin="SK"/>
