File: Hardware/Eagle files/Smart ezNODE 503 guide lines.brd (EAGLE design)
At the start: 97.2 x 63.4 mm, 18 parts, among them X1 SSW-114-02-S-D-DH, X2 SSW-114-02-S-D-DV, X3 SSW-114-02-S-D-DV, X4 SSW-114-02-S-D-DH

Commit message: Add files via upload
Connections:
- net VCC33: no longer PWS1.5
Changed lines of the file:
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@@
 <setting verticaltext="up"/>
 </settings>
-<grid distance="0.125" unitdist="mm" unit="mm" style="lines" multiple="1" display="yes" altdistance="0.025" altunitdist="inch" altunit="inch"/>
+<grid distance="0.5" unitdist="mm" unit="mm" style="lines" multiple="1" display="yes" altdistance="0.025" altunitdist="inch" altunit="inch"/>
 <layers>
 <layer number="1" name="Top" color="4" fill="1" visible="yes" active="yes"/>
@@
 <contactref element="X1" pad="2"/>
 <contactref element="X1" pad="1"/>
-<contactref element="PWS1" pad="5"/>
 <contactref element="X4" pad="2"/>
 <contactref element="X4" pad="1"/>
@@
 <contactref element="WMOD_OPZ" pad="1"/>
 <contactref element="ICP" pad="2"/>
-<wire x1="75.73" y1="29.2" x2="74.04" y2="39.04" width="0" layer="19" extent="16-16"/>
-<wire x1="78.27" y1="29.2" x2="75.73" y2="29.2" width="0" layer="19" extent="16-16"/>
+<wire x1="75.73" y1="29.2" x2="78.27" y2="29.2" width="0" layer="19" extent="16-16"/>
 <wire x1="60.2" y1="29.2" x2="75.73" y2="29.2" width="0" layer="19" extent="16-16"/>
 <wire x1="56.2" y1="29.2" x2="60.2" y2="29.2" width="0" layer="19" extent="16-16"/>
-<wire x1="41" y1="18.8" x2="56.2" y2="29.2" width="0" layer="19" extent="16-16"/>
+<wire x1="45.25" y1="34.24" x2="56.2" y2="29.2" width="0" layer="19" extent="16-16"/>
+<wire x1="41" y1="18.8" x2="45.25" y2="34.24" width="0" layer="19" extent="16-16"/>
 <wire x1="37" y1="18.8" x2="41" y2="18.8" width="0" layer="19" extent="16-16"/>
 <wire x1="31.06" y1="20.3" x2="37" y2="18.8" width="0" layer="19" extent="16-16"/>
@@
 <wire x1="22.2" y1="40" x2="31.06" y2="22.84" width="0" layer="19" extent="16-16"/>
 <wire x1="3.1" y1="54" x2="22.2" y2="40" width="0" layer="19" extent="16-16"/>
-<wire x1="45.25" y1="34.24" x2="19.03" y2="18.8" width="0" layer="19" extent="1-16"/>
 </signal>
 <signal name="CS_DIS">
@@
 <polygon width="0.254" layer="1" pour="cutout" thermals="no">
 <vertex x="85.5" y="24.375"/>
-<vertex x="85.5" y="47"/>
-<vertex x="97" y="47"/>
+<vertex x="85.5" y="62.5"/>
+<vertex x="97" y="62.5"/>
 <vertex x="97" y="24.375"/>
 </polygon>
@@
 <signal name="N$3">
 <polygon width="0.254" layer="16" pour="cutout">
-<vertex x="85.5" y="47"/>
-<vertex x="97" y="47"/>
+<vertex x="85.5" y="62.5"/>
+<vertex x="97" y="62.5"/>
 <vertex x="97" y="24.375"/>
 <vertex x="85.5" y="24.375"/>
