File: Hardware/Eagle files/Smart ezNODE 503 guide lines.sch (EAGLE design)
At the start: 18 parts, among them X1 SSW-114-02-S-D-DH, X2 SSW-114-02-S-D-DV, X3 SSW-114-02-S-D-DV, X4 SSW-114-02-S-D-DH

Commit message: Add files via upload
Connections:
- net VCC33: no longer PWS1.+VOUT1
Changed lines of the file:
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@@
 <setting verticaltext="up"/>
 </settings>
-<grid distance="0.1" unitdist="inch" unit="inch" style="lines" multiple="1" display="no" altdistance="0.01" altunitdist="inch" altunit="inch"/>
+<grid distance="0.05" unitdist="inch" unit="inch" style="lines" multiple="1" display="yes" altdistance="0.01" altunitdist="inch" altunit="inch"/>
 <layers>
 <layer number="1" name="Top" color="4" fill="1" visible="no" active="no"/>
@@
 <attribute name="NAME" x="83.312" y="38.862" size="1.524" layer="95" rot="R180"/>
 </instance>
-<instance part="SUPPLY1" gate="1" x="303.53" y="213.36" rot="MR0"/>
+<instance part="SUPPLY1" gate="1" x="293.37" y="213.36" rot="MR0"/>
 <instance part="SUPPLY2" gate="1" x="331.47" y="33.02" rot="MR0"/>
 <instance part="SUPPLY3" gate="1" x="293.37" y="33.02" rot="MR0"/>
@@
 <segment>
 <pinref part="PWS1" gate="G$1" pin="COM"/>
-<wire x1="308.61" y1="218.44" x2="303.53" y2="218.44" width="0.1524" layer="91"/>
-<wire x1="303.53" y1="218.44" x2="303.53" y2="215.9" width="0.1524" layer="91"/>
+<wire x1="308.61" y1="218.44" x2="293.37" y2="218.44" width="0.1524" layer="91"/>
+<wire x1="293.37" y1="218.44" x2="293.37" y2="215.9" width="0.1524" layer="91"/>
 <pinref part="SUPPLY1" gate="1" pin="GND"/>
 </segment>
@@
 </segment>
 <segment>
-<pinref part="PWS1" gate="G$1" pin="+VOUT1"/>
-<wire x1="308.61" y1="220.98" x2="303.53" y2="220.98" width="0.1524" layer="91"/>
-<label x="300.99" y="220.98" size="1.27" layer="95" rot="MR0"/>
-</segment>
-<segment>
 <wire x1="326.39" y1="71.12" x2="331.47" y2="71.12" width="0.1524" layer="91"/>
 <label x="334.01" y="71.12" size="1.27" layer="95"/>
@@
 <wire x1="203.2" y1="143.51" x2="205.74" y2="143.51" width="0.1524" layer="91"/>
 </segment>
+<segment>
+<wire x1="308.61" y1="215.9" x2="303.53" y2="215.9" width="0.1524" layer="91"/>
+<label x="295.91" y="215.9" size="1.27" layer="95"/>
+</segment>
 </net>
