File: Hardware/Eagle files/Smart ezNODE 503 M1.brd (EAGLE design)
At the start: 97.2 x 63.4 mm, 30 parts, among them IC1 FT232RLSSOP, IC2 NLAS4684, SW1 SLIDE_SWITCH_2P_2W_ALPS, SW2 SLIDE_SWITCH_3P_2W_ALPS, X1 MINI-USB-SCHIELD, X2 SSW-114-02-S-D-DH

Commit message: Add files via upload
Parts:
- IC1: value FT232RLSSOP -> FT232R-QFN32; device Multiconnect_base:SSOP28DB -> Multiconnect_base:QFN32
- moved C1 13.4 mm to (8.00, 3.00)
- moved C2 12.2 mm to (18.0, 3.00)
- moved IC1 2.69 mm to (12.0, 9.00), turned to 0 degrees
- moved C5 2.06 mm to (8.00, 15.5)
- moved IC2 2.06 mm to (12.0, 15.5)
- moved C6 1.12 mm to (26.8, 3.75)
- moved C7 1.12 mm to (26.8, 2.25)
- moved XTAL1 1.12 mm to (25.0, 3.00)
- moved C4 1.00 mm to (26.5, 9.00)
- moved MCU 1.00 mm to (20.5, 9.00)
- moved C3 0.50 mm to (24.5, 33.5)
- moved R1 0.50 mm to (6.00, 33.5)
- moved R2 0.50 mm to (8.00, 33.5)
- moved R3 0.50 mm to (12.0, 33.5)
- moved R4 0.50 mm to (16.0, 33.5)
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Connections:
- net D+: now also IC1.14; no longer IC1.15
- net D-: now also IC1.15; no longer IC1.16
- net GND: now also IC1.17, IC1.20, IC1.24, IC1.4, IC1.EXP; no longer IC1.18, IC1.21, IC1.25, IC1.7
- net N$6: now also IC1.1, IC1.16; no longer IC1.17, IC1.4
- net RESET: now also IC1.18
- net RXD_USB: now also IC1.2; no longer IC1.5
- net TXD_USB: now also IC1.30; no longer IC1.1
- net VBUS: now also IC1.19; no longer IC1.20
Routing:
- net WMOD_TXD-->RXD_USB: track 48.7 -> 91.1 mm, vias 3 -> 5
- net GND: track 183.1 -> 220.3 mm, vias 8 -> 13
- net MCU_(D7): track 62.1 -> 36.5 mm
- net WMOD_RXD<--TXD_USB: track 71.7 -> 47.7 mm, vias 7 -> 3
- net RESET: track 89.7 -> 112.2 mm, vias 6 -> 7
- net SCK: track 85.9 -> 104.2 mm
- net MISO: track 99.4 -> 83.7 mm, vias 10 -> 9
- net MCU_(D5): track 21.2 -> 36.2 mm, vias 2 -> 4
- net ZB/SX_RXD<--TXD: track 42.8 -> 57.0 mm, vias 2 -> 3
- net ZB/SX_TXD-->RXD: track 48.4 -> 61.6 mm, vias 2 -> 5
- net MCU_(D10): track 52.0 -> 64.4 mm, vias 7 -> 9
- net MCU_(D3): track 12.2 -> 23.9 mm, vias 2 -> 4
- net N$1: track 8.43 -> 19.5 mm, vias 3 -> 5
- net SCL: track 84.0 -> 94.2 mm, vias 6 -> 8
- net CS_SD: track 23.5 -> 32.0 mm, vias 1 -> 5
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