File: Hardware/Eagle files/Smart ezNODE 503 M1.sch (EAGLE design)
At the start: 30 parts, among them IC1 FT232RLSSOP, IC2 NLAS4684, SW1 SLIDE_SWITCH_2P_2W_ALPS, SW2 SLIDE_SWITCH_3P_2W_ALPS, X1 MINI-USB-SCHIELD, X2 SSW-114-02-S-D-DH

Commit message: Add files via upload
Parts:
- IC1: value FT232RLSSOP -> FT232R-QFN32; device Multiconnect_base:FT232RLSSOP -> Multiconnect_base:FT232R-QFN32
Connections:
- net GND: now also IC1.GND-1, IC1.GND-2, IC1.GND-3, IC1.GND_EXT; no longer IC1.GND18, IC1.GND21, IC1.GND7
- net RESET: now also IC1.RESET
Other:
- note added: "EXP GND is manualy traced on PCB out of autorouting"
