File: Hardware/Eagle files/Smart ezNODE 503 M2.brd (EAGLE design)
At the start: 97.2 x 63.4 mm, 26 parts, among them IC1 DS133X, X1 SSW-114-02-S-D-DV, X2 SSW-114-02-S-D-DV

Commit message: Add files via upload
Routing:
- net S3: track 67.6 -> 143.5 mm, vias 4 -> 6
- net NC3: track 21.9 -> 68.6 mm
- net S2: track 56.0 -> 101.0 mm, vias 3 -> 4
- net SCL: track 109.9 -> 75.0 mm, vias 6 -> 4
- net MCU_(A0): track 31.9 -> 64.2 mm
- net MCU_(D10): track 64.8 -> 38.4 mm, vias 2 -> 4
- net MCU_(D3): track 51.4 -> 30.5 mm, vias 4 -> 2
- net SCK: track 62.4 -> 46.9 mm, vias 4 -> 6
- net CS_DIS_MCU: track 63.8 -> 49.5 mm, vias 2 -> 8
- net VCC33: track 148.8 -> 135.6 mm, vias 7 -> 5
- net NC2: track 18.5 -> 30.9 mm, vias 2 -> 4
- net GND: track 215.6 -> 204.5 mm
- net NC1: track 55.7 -> 46.0 mm
- net WMOD_(D15): track 32.6 -> 23.1 mm
- net MCU_(D2): track 48.6 -> 41.3 mm
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